File: keyboard/keyboard.kicad_pcb (KiCad board)
At the start: 2 copper layers, 88 parts

Commit message: ~finished schematic, started layout
Parts:
- added C1: 10uf, Capacitor_SMD:C_0805_2012Metric_Pad1.18x1.45mm_HandSolder, F.Cu at (151.7, 20.3)
- added C2: 1uf, Capacitor_SMD:C_0805_2012Metric_Pad1.18x1.45mm_HandSolder, F.Cu at (151.7, 23.3)
- added C3: 10uf, Capacitor_SMD:C_0805_2012Metric_Pad1.18x1.45mm_HandSolder, F.Cu at (151.7, 26.3)
- added C4: 10uf, Capacitor_SMD:C_0805_2012Metric_Pad1.18x1.45mm_HandSolder, F.Cu at (151.7, 29.4)
- added C5: 100nf, Capacitor_SMD:C_0805_2012Metric_Pad1.18x1.45mm_HandSolder, F.Cu at (151.7, 32.4)
- added D1: CHRG_LED, LED_SMD:LED_0805_2012Metric_Pad1.15x1.40mm_HandSolder, F.Cu at (146.9, 20.3)
- added D2: LED, LED_SMD:LED_0805_2012Metric_Pad1.15x1.40mm_HandSolder, F.Cu at (146.9, 23.4)
- added D3: LED, LED_SMD:LED_0805_2012Metric_Pad1.15x1.40mm_HandSolder, F.Cu at (146.9, 26.4)
- added D4: LED, LED_SMD:LED_0805_2012Metric_Pad1.15x1.40mm_HandSolder, F.Cu at (146.9, 29.5)
- added D5: LED, LED_SMD:LED_0805_2012Metric_Pad1.15x1.40mm_HandSolder, F.Cu at (146.9, 32.5)
- added IC2: NPM1300-QEAA-R7, mylib:QFN50P500X500X90-33N, F.Cu at (157.7, 31.3)
- added J1: PROG, mylib:SWD_PROG_5pin, F.Cu at (166.4, 53.3)
- added J10: Conn_01x01, Connector_Wire:SolderWirePad_1x01_SMD_1x2mm, F.Cu at (151.4, 2.75)
- added J11: Conn_01x01, Connector_Wire:SolderWirePad_1x01_SMD_1x2mm, F.Cu at (151.4, 7.34)
- added J12: Conn_01x01, Connector_Wire:SolderWirePad_1x01_SMD_1x2mm, F.Cu at (151.4, 11.9)
- added J13: Conn_01x01, Connector_Wire:SolderWirePad_1x01_SMD_1x2mm, F.Cu at (151.4, 16.5)
- added J14: Conn_01x01, Connector_Wire:SolderWirePad_1x01_SMD_1x2mm, F.Cu at (156.0, -1.84)
- added J15: Conn_01x01, Connector_Wire:SolderWirePad_1x01_SMD_1x2mm, F.Cu at (156.0, 2.75)
- added J16: Conn_01x01, Connector_Wire:SolderWirePad_1x01_SMD_1x2mm, F.Cu at (156.0, 7.34)
- added J17: Conn_01x01, Connector_Wire:SolderWirePad_1x01_SMD_1x2mm, F.Cu at (156.0, 11.9)
- added J18: Conn_01x01, Connector_Wire:SolderWirePad_1x01_SMD_1x2mm, F.Cu at (156.0, 16.5)
- added J19: Conn_01x01, Connector_Wire:SolderWirePad_1x01_SMD_1x2mm, F.Cu at (160.6, -1.84)
- added J2: disp, Connector_PinHeader_2.54mm:PinHeader_1x04_P2.54mm_Vertical, F.Cu at (154.0, 79.5)
- added J20: Conn_01x01, Connector_Wire:SolderWirePad_1x01_SMD_1x2mm, F.Cu at (160.6, 2.75)
- added J21: Conn_01x01, Connector_Wire:SolderWirePad_1x01_SMD_1x2mm, F.Cu at (160.6, 7.34)
- added J22: Conn_01x01, Connector_Wire:SolderWirePad_1x01_SMD_1x2mm, F.Cu at (160.6, 11.9)
- added J3: BAT, Connector_PinHeader_2.54mm:PinHeader_1x02_P2.54mm_Vertical, B.Cu at (105.0, 52.0)
- added J4: Conn_01x01, Connector_Wire:SolderWirePad_1x01_SMD_1x2mm, F.Cu at (146.8, -1.84)
- added J5: Conn_01x01, Connector_Wire:SolderWirePad_1x01_SMD_1x2mm, F.Cu at (146.8, 2.75)
- added J6: Conn_01x01, Connector_Wire:SolderWirePad_1x01_SMD_1x2mm, F.Cu at (146.8, 7.34)
- added J7: Conn_01x01, Connector_Wire:SolderWirePad_1x01_SMD_1x2mm, F.Cu at (146.8, 11.9)
- added J8: Conn_01x01, Connector_Wire:SolderWirePad_1x01_SMD_1x2mm, F.Cu at (146.8, 16.5)
- added J9: Conn_01x01, Connector_Wire:SolderWirePad_1x01_SMD_1x2mm, F.Cu at (151.4, -1.84)
- added L1: L, Inductor_SMD:L_1008_2520Metric_Pad1.43x2.20mm_HandSolder, F.Cu at (164.0, 34.2)
- added Q1: FS8205A, FS8205A:SOP65P640X120-8N, B.Cu at (111.0, 52.5)
- added R1: 300k, Resistor_SMD:R_0805_2012Metric_Pad1.20x1.40mm_HandSolder, F.Cu at (165.2, -2.66)
- added R2: 1K, Resistor_SMD:R_0805_2012Metric_Pad1.20x1.40mm_HandSolder, F.Cu at (165.2, 0.29)
- added R3: 100R, Resistor_SMD:R_0805_2012Metric_Pad1.20x1.40mm_HandSolder, F.Cu at (165.2, 3.24)
- added R4: 1k, Resistor_SMD:R_0805_2012Metric_Pad1.20x1.40mm_HandSolder, F.Cu at (165.2, 6.19)
- added R5: 1k, Resistor_SMD:R_0805_2012Metric_Pad1.20x1.40mm_HandSolder, F.Cu at (165.2, 9.14)
- added R6: 1k, Resistor_SMD:R_0805_2012Metric_Pad1.20x1.40mm_HandSolder, F.Cu at (165.2, 12.1)
- added R7: 1k, Resistor_SMD:R_0805_2012Metric_Pad1.20x1.40mm_HandSolder, F.Cu at (165.2, 15.0)
- added U1: ~, mylib:nrf54l15_holyiot, B.Cu at (150.3, 60.0)
- added U2: DW01A, Package_TO_SOT_SMD:SOT-23-6, B.Cu at (111.1, 49.0)
- added U3: USBC20, my_usbc:USBC_6PIN, B.Cu at (190.5, 46.8)
Connections:
- D5:0 pad 1: Net-(D0:2-K) -> SHPHLD
- SW5:0 pad 1: Net-(SW5:0-a) -> SHPHLD
- SW5:0 pad 2: Net-(D5:0-A) -> Net-(D0:2-K)
- SW5:1 pad 1: Net-(SW5:0-a) -> Net-(D5:0-A)
- SW6:0 pad 2: Net-(SW5:0-a) -> Net-(D5:0-A)
- SW6:1 pad 2: Net-(SW5:0-a) -> Net-(D5:0-A)
Routing:
- net Net-(J3-Pin_1): track 0.00 -> 11.5 mm
- net Net-(U2-OD): track 0.00 -> 6.41 mm
- net Net-(U2-OC): track 0.00 -> 2.29 mm
- net GND: track 0.00 -> 0.65 mm

Commit message: v1.0 PCB (jlcpcb order)
Parts:
- removed J19, J20, J21, J22, J4, J5, J6, J7, J8: Conn_01x01, Connector_Wire:SolderWirePad_1x01_SMD_1x2mm
- added H1: MountingHole_Pad, MountingHole:MountingHole_2.2mm_M2_DIN965_Pad, F.Cu at (247.5, 120.5)
- added H2: MountingHole_Pad, MountingHole:MountingHole_2.2mm_M2_DIN965_Pad, F.Cu at (52.5, 120.5)
- added H3: MountingHole_Pad, MountingHole:MountingHole_2.2mm_M2_DIN965_Pad, F.Cu at (150.0, 127.0)
- added H4: MountingHole_Pad, MountingHole:MountingHole_2.2mm_M2_DIN965_Pad, F.Cu at (150.0, 103.0)
- added H5: MountingHole_Pad, MountingHole:MountingHole_2.2mm_M2_DIN965_Pad, F.Cu at (167.0, 82.0)
- added H6: MountingHole_Pad, MountingHole:MountingHole_2.2mm_M2_DIN965_Pad, F.Cu at (142.0, 72.0)
- added H7: MountingHole_Pad, MountingHole:MountingHole_2.2mm_M2_DIN965_Pad, F.Cu at (219.0, 48.0)
- added H8: MountingHole_Pad, MountingHole:MountingHole_2.2mm_M2_DIN965_Pad, F.Cu at (80.5, 48.0)
- added R8: 0R, Resistor_SMD:R_0805_2012Metric_Pad1.20x1.40mm_HandSolder, F.Cu at (136.0, 92.0)
- Q1, U1, U2, U3: moved to F.Cu
- moved D2:0 110.4 mm to (98.5, 55.5), turned to 80 degrees
- moved R2 82.0 mm to (100.5, 50.6), turned to 90 degrees
- moved R3 73.0 mm to (108.0, 48.5), turned to 90 degrees
- moved J14 72.5 mm to (119.0, 60.5)
- moved J9 70.8 mm to (143.0, 68.5), turned to 90 degrees
- moved J15 67.5 mm to (121.0, 60.5)
- moved R1 67.4 mm to (129.5, 54.5)
- moved J10 64.8 mm to (143.0, 67.0), turned to 90 degrees
- moved J16 62.5 mm to (123.0, 60.5)
- moved J11 58.8 mm to (143.0, 65.5), turned to 90 degrees
- moved J17 57.4 mm to (121.0, 57.5)
- moved J18 55.2 mm to (119.0, 57.5)
- moved J12 51.8 mm to (143.0, 63.0), turned to 90 degrees
- moved U3 51.0 mm to (139.5, 47.5), turned to 180 degrees
- moved L1 49.7 mm to (117.1, 50.6), turned to 90 degrees
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Connections:
- C3 pad 2: 3V3 -> GND
- D5:0 pad 1: SHPHLD -> Net-(D5:0-K)
- IC2 pad 15: SHPHLD -> Net-(IC2-SHPHLD)
- IC2 pad 26: Net-(IC2-LED1) -> unconnected-(IC2-LED1-Pad26)
- IC2 pad 27: Net-(IC2-LED2) -> unconnected-(IC2-LED2-Pad27)
- IC2 pad 30: Net-(IC2-LSIN2/VINLDO2) -> unconnected-(IC2-LSIN2/VINLDO2-Pad30)
- IC2 pad 31: Net-(IC2-LSOUT2/VOUTLDO2) -> unconnected-(IC2-LSOUT2/VOUTLDO2-Pad31)
- SW5:0 pad 1: SHPHLD -> Net-(D5:0-K)
- SW5:0 pad 2: Net-(D0:2-K) -> GND
- SW5:1 pad 1: Net-(D5:0-A) -> Net-(SW5:1-a)
- SW6:0 pad 2: Net-(D5:0-A) -> Net-(SW5:1-a)
- SW6:1 pad 2: Net-(D5:0-A) -> Net-(SW5:1-a)
- U1 pad 22: Net-(D5:0-A) -> Net-(SW5:1-a)
- U1 pad 28: Net-(J8-Pin_1) -> Net-(D0:0-K)
- U1 pad 29: Net-(J7-Pin_1) -> Net-(D0:1-K)
- U1 pad 32: Net-(J6-Pin_1) -> Net-(D0:2-K)
- U1 pad 33: Net-(J5-Pin_1) -> Net-(D0:3-K)
- U1 pad 34: Net-(J4-Pin_1) -> Net-(D5:0-A)
Routing:
- net Net-(D0:3-K): track 0.00 -> 329.5 mm, vias 0 -> 13
- net Net-(D0:1-K): track 0.00 -> 307.9 mm, vias 0 -> 12
- net Net-(D0:2-K): track 0.00 -> 306.9 mm, vias 0 -> 10
- net Net-(D0:0-K): track 0.00 -> 276.0 mm, vias 0 -> 13
- net Net-(SW0:0-a): track 0.00 -> 185.8 mm, vias 0 -> 1
- net Net-(SW1:0-a): track 0.00 -> 165.6 mm, vias 0 -> 1
- net Net-(SW11:0-b): track 0.00 -> 156.1 mm, vias 0 -> 1
- net 3V3: track 0.00 -> 155.5 mm, vias 0 -> 6
- net Net-(SW2:0-a): track 0.00 -> 147.2 mm, vias 0 -> 1
- net Net-(SW10:0-b): track 0.00 -> 135.8 mm, vias 0 -> 1
- net Net-(SW3:0-a): track 0.00 -> 131.4 mm, vias 0 -> 1
- net Net-(SW9:0-b): track 0.00 -> 119.4 mm, vias 0 -> 1
- net Net-(SW4:0-a): track 0.00 -> 112.7 mm, vias 0 -> 1
- net Net-(SW5:1-a): track 0.00 -> 103.3 mm
- net GND: track 0.65 -> 103.4 mm, vias 0 -> 25
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- added copper zone on B.Cu, net GND
- added copper zone on F.Cu, net GND
Other:
- board outline added: 237.1 x 92.5 mm
- board text added: "B+"
- board text added: "B-"
- board text added: "PK 2025"
- board text added: "wrls_atreus v1.0"
